File: pulse_generator.kicad_pcb (KiCad board)
At the start: 4 copper layers, 82.6 x 53 mm, 29 parts, among them J1 Power, J2 Digital/PWM, J3 Analog, J4 Digital/PWM, J5 Conn_Coaxial, J6 Conn_Coaxial, SW1 SW_Push, U1 LM311, U2 74LS279

Commit message: minor tweaks
Other:
- board text added: "GND"
- board text added: "Keystone test loops or similar"
- board text added: "ø1.5"
Changed lines of the file:
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@@
     (fp_line (start 1.27 1.27) (end -1.27 1.27)
       (stroke (width 0.1) (type solid)) (layer "F.Fab"))
-    (pad "1" thru_hole rect (at 0 0) (size 1.7 1.7) (drill 1) (layers "*.Cu" "*.Mask")
+    (pad "1" thru_hole rect (at 0 0) (size 2 2) (drill 1.3) (layers "*.Cu" "*.Mask")
       (net 5 "/A0") (pinfunction "1") (pintype "passive"))
     (model "${KICAD6_3DMODEL_DIR}/Connector_PinHeader_2.54mm.3dshapes/PinHeader_1x01_P2.54mm_Vertical.wrl"
@@
     (property "Sheetname" "")
     (attr through_hole)
-    (fp_text reference "U2" (at 3.81 -2.33 -90) (layer "F.SilkS")
+    (fp_text reference "U2" (at 4.12 17.24 -90) (layer "F.SilkS")
         (effects (font (size 1 1) (thickness 0.15)))
     )
@@
         (effects (font (size 1 1) (thickness 0.15)))
     )
-    (fp_text value "GND_hook" (at 0 2.5) (layer "F.SilkS")
+    (fp_text value "GND_hook" (at 0 2.5) (layer "F.Fab")
         (effects (font (size 1 1) (thickness 0.15)))
     )
@@
     (fp_line (start 1.27 1.27) (end -1.27 1.27)
       (stroke (width 0.1) (type solid)) (layer "F.Fab"))
-    (pad "1" thru_hole rect (at 0 0) (size 1.7 1.7) (drill 1) (layers "*.Cu" "*.Mask")
+    (pad "1" thru_hole rect (at 0 0) (size 2 2) (drill 1.3) (layers "*.Cu" "*.Mask")
       (net 1 "GND") (pinfunction "1") (pintype "passive"))
     (model "${KICAD6_3DMODEL_DIR}/Connector_PinHeader_2.54mm.3dshapes/PinHeader_1x01_P2.54mm_Vertical.wrl"
@@
     (effects (font (size 1 1) (thickness 0.15)) (justify left bottom))
   )
+  (gr_text "ø1.5" (at 138.5 95.5) (layer "F.SilkS")
+    (effects (font (size 1 1) (thickness 0.15)) (justify left bottom))
+  )
   (gr_text "Pull-up" (at 123.5 75) (layer "F.SilkS")
     (effects (font (size 1 1) (thickness 0.15)) (justify right bottom))
@@
     (effects (font (size 1 1) (thickness 0.15)) (justify left bottom))
   )
+  (gr_text "GND" (at 137.5 87.5) (layer "F.SilkS")
+    (effects (font (size 1 1) (thickness 0.15)) (justify left bottom))
+  )
   (gr_text "R1" (at 151.5 92.5) (layer "F.SilkS")
     (effects (font (size 1 1) (thickness 0.15)) (justify left bottom))
@@
     (effects (font (size 1 1) (thickness 0.15)) (justify left bottom))
   )
+  (gr_text "Keystone test \nloops or similar" (at 126 95.5) (layer "F.SilkS")
+    (effects (font (size 1 1) (thickness 0.15)) (justify left bottom))
+  )

Commit message: Added all assets and 3d models
Other:
- board text added: "CC-BY-SA 2023"
Changed lines of the file:
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@@
   (gr_rect (start 115 70.5) (end 131.5 76)
     (stroke (width 0.15) (type default)) (fill none) (layer "F.SilkS"))
-  (gr_rect (start 86 47.8) (end 96 54.3)
+  (gr_rect (start 86 48.05) (end 96 54.05)
     (stroke (width 0.15) (type solid)) (fill none) (layer "F.SilkS"))
   (gr_poly
@@
     (effects (font (size 1 1) (thickness 0.15)) (justify left bottom))
   )
+  (gr_text "CC-BY-SA 2023" (at 98 50.5) (layer "F.SilkS")
+    (effects (font (size 1 1) (thickness 0.15)) (justify left bottom))
+  )

Commit message: corrected some stuff, larger enclosure
Parts:
- added R8: 0, Resistor_SMD:R_0805_2012Metric_Pad1.20x1.40mm_HandSolder, F.Cu at (106.0, 93.5)
- added R9: 0, Resistor_SMD:R_0805_2012Metric_Pad1.20x1.40mm_HandSolder, F.Cu at (106.0, 68.5)
- moved C1 3.94 mm to (145.5, 69.0)
- moved R6 0.50 mm to (106.0, 60.0)
Connections:
- J5 pad 2: GND -> Net-(J5-Ext)
- J6 pad 2: GND -> Net-(J6-Ext)
Routing:
- net GND: track 11.0 -> 14.9 mm, vias 7 -> 9
- net /~{RESET}: track 60.1 -> 58.0 mm
- net Net-(J6-Ext): track 0.00 -> 1.50 mm, vias 0 -> 1
- net Net-(J5-Ext): track 0.00 -> 1.50 mm, vias 0 -> 1
- net Net-(D5-K): track 12.9 -> 12.4 mm
- added copper zone on In1.Cu, net Net-(J5-Ext)
- added copper zone on In1.Cu, net Net-(J6-Ext)
Other:
- board text added: "0805"
- board text added: "0R"
- board text added: "All passives are and up"
- board text added: "R9/R8 disconnect BNC shield from GND"
