File: hardware/pulse_generator.kicad_sch (KiCad schematic)
At the start: 27 parts, among them J1 Power, J2 Digital/PWM, J3 Analog, J4 Digital/PWM, J5 Conn_Coaxial, J6 Conn_Coaxial, SW1 SW_Push, U1 LM311, U2 74LS279

Commit message: some changes related to testing
Other:
- note added: "bruh"
Changed lines of the file:
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@@
     (stroke (width 0) (type solid))
+  )
+  (circle (center 127 38.1) (radius 4.0161)
+    (stroke (width 0) (type default))
+    (fill (type none))
+  )
+  (text "bruh" (at 129.54 43.18 0)
+    (effects (font (size 1.27 1.27)) (justify left bottom))
   )
   (text "* Indicates a PWM-capable pin" (at 92.71 118.11 0)
