File: hardware/v2/board/pulse_generator_v2.kicad_pcb (KiCad board)
At the start: 4 copper layers, 82.6 x 62.5 mm, 51 parts, among them J1 Power, J2 Digital/PWM, J3 Analog, J4 Digital/PWM, J5 Conn_Coaxial, J6 Conn_Coaxial, K1 G6K-2, Q1 BC337, Q2 BC337, Q3 BC337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

Commit message: gerbers out
Parts:
- added TP5: GND_pad, TestPoint:TestPoint_Pad_2.5x2.5mm, F.Cu at (107.0, 97.8)
- moved R4 2.51 mm to (106.8, 57.0)
- moved C3 0.50 mm to (122.0, 80.5)
- moved J5 0.20 mm to (98.6, 91.5)
- moved J6 0.20 mm to (98.6, 66.5)
Routing:
- net GND: track 15.9 -> 19.7 mm
- net Net-(D6-A): track 40.6 -> 42.2 mm
- net Net-(D3-A): track 18.7 -> 17.2 mm
- net /~{RESET}: track 121.6 -> 120.7 mm
Other:
- board text added: "10u"
- board text added: "J5/J6: Amphenol B6252H7-NPP3G-50 or matching BNC"
- board text added: "TPx: RSPRO 262-2034 test loops or similar. ø1mm"
- board text removed: "J5/J6: Amphenol B6252H5-NPP3G-50 or matching BNC"
- board text removed: "OJO: LORDRE DELS LEDS HA CANVIAT MIRAR LLIBRETA"
- board text removed: "TPx: Keystone test loops or similar ø1.5mm"
