File: hardware/v2/board/pulse_generator_v2.kicad_sch (KiCad schematic)
At the start: 47 parts, among them J1 Power, J2 Digital/PWM, J3 Analog, J4 Digital/PWM, J5 Conn_Coaxial, J6 Conn_Coaxial, K1 G6K-2, Q1 BC337, Q2 BC337, Q3 BC337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

Commit message: gerbers out
Parts:
- added TP5: GND_pad, TestPoint:TestPoint_Pad_2.5x2.5mm, symbol Connector:TestPoint
Connections:
- net GND: now also TP5.1
Other:
- note added: "DECOUPLING"
Changed lines of the file:
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@@
   (junction (at 166.37 114.3) (diameter 0) (color 0 0 0 0)
+  )
+  (junction (at 41.91 137.16) (diameter 0) (color 0 0 0 0)
   )
   (junction (at 39.37 80.01) (diameter 0) (color 0 0 0 0)
@@
     (stroke (width 0) (type solid))
   )
+  (wire (pts (xy 41.91 137.16) (xy 49.53 137.16))
+    (stroke (width 0) (type default))
+  )
   (wire (pts (xy 49.53 132.08) (xy 52.07 132.08))
     (stroke (width 0) (type solid))
@@
     (stroke (width 0) (type default))
   )
-  (wire (pts (xy 39.37 137.16) (xy 49.53 137.16))
+  (wire (pts (xy 39.37 137.16) (xy 41.91 137.16))
     (stroke (width 0) (type default))
   )
@@
     (stroke (width 0) (type default))
   )
+  (wire (pts (xy 41.91 135.89) (xy 41.91 137.16))
+    (stroke (width 0) (type default))
+  )
   (wire (pts (xy 34.29 64.77) (xy 39.37 64.77))
     (stroke (width 0) (type default))
@@
   )
   (rectangle (start 20.32 104.14) (end 107.95 177.8)
+    (stroke (width 0) (type default))
+    (fill (type none))
+  )
+  (rectangle (start 114.3 146.05) (end 140.97 177.8)
     (stroke (width 0) (type default))
     (fill (type none))
@@
   (text "SET" (at 93.98 160.02 0)
     (effects (font (size 1.27 1.27)) (justify left bottom))
+  )
+  (text "DECOUPLING" (at 115.57 144.78 0)
+    (effects (font (size 1.27 1.27) (thickness 0.254) bold) (justify left bottom))
   )
   (text "BACKLIGHT" (at 115.57 102.87 0)
@@
         )
       )
+    )
+  )
+  (symbol (lib_id "Connector:TestPoint") (at 41.91 135.89 0) (unit 1)
+    (in_bom yes) (on_board yes) (dnp no)
+    (property "Reference" "TP5" (at 39.37 130.81 0)
+      (effects (font (size 1.27 1.27)) (justify left))
+    )
+    (property "Value" "GND_pad" (at 34.29 139.7 0)
+      (effects (font (size 1.27 1.27)) (justify left))
+    )
+    (property "Footprint" "TestPoint:TestPoint_Pad_2.5x2.5mm" (at 46.99 135.89 0)
+      (effects (font (size 1.27 1.27)) hide)
+    )
+    (property "Datasheet" "~" (at 46.99 135.89 0)
+      (effects (font (size 1.27 1.27)) hide)
+    )
+    (pin "1")
+    (instances
+      (project "pulse_generator_v2"
+        (path "/e63e39d7-6ac0-4ffd-8aa3-1841a4541b55"
+          (reference "TP5") (unit 1)
+        )
+      )
