File: hardware/v2/endplate/pulse_generator_endplate_v2.kicad_pcb (KiCad board)
At the start: 2 copper layers, 103 x 53 mm, 1 part, among them J2 Conn_01x01_Pin

Commit message: gerbers out
Other:
- board text added: "5Vpp"
- board text added: "5Vpp MAX"
- board text added: "Endplate version 2 Designed for 11mm standoffs between the nucleo and the ablator interface PCB. BNCs are B6252H7-NPP3G-50 Grounding post is Hirschmann 930103188 When fully assembled, J2 is connected to the enclosure. If necessary it can be used to modwire a shunt to TP5 on the ablator interface PCB."
- board text removed: "Endplate version 2 Designed for 11mm standoffs between the nucleo and the shield. BNCs are B6252H7-NPP3G-50 Grounding post is Hirschmann 930103188 When fully assembled, J2 is connected to the enclosure."
